File: pcb/pet on a chip/pet on a chip.kicad_sch (KiCad schematic)
At the start: 39 parts, among them J1 USB_B, J2 Screw_Terminal_01x02, U1 93LCxxC, U2 FT2232HL, U3 LDL1117S33R, U4 TLV70012DDCR, X1 ASTX-H11

Commit message: cleaned up kicad stuff
Other:
- sheet FPGA renamed fpga
- sheet fpga: file FPGA.kicad_sch -> fpga.kicad_sch
Changed lines of the file:
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@@
     (stroke (width 0) (type solid) (color 0 0 0 0))
     (fill (color 0 0 0 0.0000))
-    (property "Sheet name" "FPGA" (id 0) (at 289.56 109.7784 0)
+    (property "Sheet name" "fpga" (id 0) (at 289.56 109.7784 0)
       (effects (font (size 1.27 1.27)) (justify left bottom))
     )
-    (property "Sheet file" "FPGA.kicad_sch" (id 1) (at 289.56 131.3946 0)
+    (property "Sheet file" "fpga.kicad_sch" (id 1) (at 289.56 131.3946 0)
       (effects (font (size 1.27 1.27)) (justify left top))
     )
